File: simmevator_pcb/simmevator_pcb.kicad_sch (KiCad schematic)
At the start: 3 parts, among them J1 PWR_IN, J2 BUCKREG, U1 XIAO-ESP32-S3-SMD

Commit message: Transmitter schematic: divider, buck header, BMP390 header
Reviewed against docs/HARDWARE.md and it matches the design:

  * R1 100k / R2 20k, tap on U1 pin 1 (D0 = GPIO1 = ADC1_CH0), R1 taken from
    the +12V net that J1 lands on, so the divider reads the pack and not the
    buck. No capacitor across R2, as designed.
  * J2 pin 3 carries +12V into the buck and pin 2 brings +5V back to U1 pin 14
    (VBUS), which is the 5V pad. U1 pin 12 (3V3_OUT) leaves the XIAO as an
    output and only feeds the BMP390 header.
  * J3 pins 3 and 4 to D5/D4 for SCL/SDA, matching platformio.ini.

Unused XIAO pads carry no-connects, so ERC stays quiet about them.

Ignores the analysis/ directory the KiCad analyzer writes.

Co-Authored-By: Claude Opus 5 <noreply@anthropic.com>
Parts:
- added J3: BMP390, Connector_PinHeader_2.54mm:PinHeader_1x07_P2.54mm_Vertical, symbol Connector_Generic:Conn_01x07
- added R1: 100k, Resistor_THT:R_Axial_DIN0207_L6.3mm_D2.5mm_P10.16mm_Horizontal, symbol Device:R
- added R2: 20k, Resistor_THT:R_Axial_DIN0207_L6.3mm_D2.5mm_P10.16mm_Horizontal, symbol Device:R
Connections:
- net +12V: now also R1.1
- net +3V3: now also J3.1 (Pin_1)
- net GND: now also J3.2 (Pin_2), R2.2
- net at U1.1 (D0): now also R1.2, R2.1
- net SDA: now reaches U1.5 (D4)
- net SDA: now also J3.4 (Pin_4)
- net SCL: now reaches U1.6 (D5)
- net SCL: now also J3.3 (Pin_3)
- no-connect marks 11 -> 22
